Commit message: refactor: proje temizliği + başlatıcı script

File: src/leo_common/leo_description/urdf/macros.xacro (robot description, xacro)
@@ -223,6 +223,6 @@
       <child link="${link_prefix}wheel_FL_link"/>
       <axis xyz="0 -1 0"/>
-      <limit effort="4.0" velocity="6.0"/>
-      <dynamics friction="0.5" damping="0.5"/>
+      <limit effort="200.0" velocity="20.0"/>
+      <dynamics friction="0.3" damping="0.3"/>
     </joint>
     <joint name="${joint_prefix}wheel_RL_joint" type="continuous">
@@ -236,6 +236,6 @@
       <child link="${link_prefix}wheel_RL_link"/>
       <axis xyz="0 -1 0"/>
-      <limit effort="4.0" velocity="6.0"/>
-      <dynamics friction="0.5" damping="0.5"/>
+      <limit effort="200.0" velocity="20.0"/>
+      <dynamics friction="0.3" damping="0.3"/>
     </joint>
     <joint name="${joint_prefix}wheel_FR_joint" type="continuous">
@@ -249,6 +249,6 @@
       <child link="${link_prefix}wheel_FR_link"/>
       <axis xyz="0 1 0"/>
-      <limit effort="4.0" velocity="6.0"/>
-      <dynamics friction="0.5" damping="0.5"/>
+      <limit effort="200.0" velocity="20.0"/>
+      <dynamics friction="0.3" damping="0.3"/>
     </joint>
     <joint name="${joint_prefix}wheel_RR_joint" type="continuous">
@@ -262,6 +262,6 @@
       <child link="${link_prefix}wheel_RR_link"/>
       <axis xyz="0 1 0"/>
-      <limit effort="4.0" velocity="6.0"/>
-      <dynamics friction="0.5" damping="0.5"/>
+      <limit effort="200.0" velocity="20.0"/>
+      <dynamics friction="0.3" damping="0.3"/>
     </joint>
     <xacro:if value="${default_antenna}">
@@ -592,8 +592,8 @@
         <odom_topic>${link_prefix}odom</odom_topic>
         <tf_topic>${link_prefix}tf</tf_topic>
-        <max_linear_acceleration>2.5</max_linear_acceleration>
-        <max_angular_acceleration>3</max_angular_acceleration>
-        <min_linear_acceleration>-2.5</min_linear_acceleration>
-        <min_angular_acceleration>-3</min_angular_acceleration>
+        <max_linear_acceleration>10.0</max_linear_acceleration>
+        <max_angular_acceleration>15.0</max_angular_acceleration>
+        <min_linear_acceleration>-10.0</min_linear_acceleration>
+        <min_angular_acceleration>-15.0</min_angular_acceleration>
       </plugin>
     </gazebo>

Commit message: Dual-UKF GPS navigasyon: 4/4 waypoint testi başarılı

File: src/leo_common/leo_description/urdf/macros.xacro (robot description, xacro)
@@ -223,6 +223,6 @@
       <child link="${link_prefix}wheel_FL_link"/>
       <axis xyz="0 -1 0"/>
-      <limit effort="200.0" velocity="20.0"/>
-      <dynamics friction="0.3" damping="0.3"/>
+      <limit effort="800.0" velocity="30.0"/>
+      <dynamics friction="1.0" damping="0.5"/>
     </joint>
     <joint name="${joint_prefix}wheel_RL_joint" type="continuous">
@@ -236,6 +236,6 @@
       <child link="${link_prefix}wheel_RL_link"/>
       <axis xyz="0 -1 0"/>
-      <limit effort="200.0" velocity="20.0"/>
-      <dynamics friction="0.3" damping="0.3"/>
+      <limit effort="800.0" velocity="30.0"/>
+      <dynamics friction="1.0" damping="0.5"/>
     </joint>
     <joint name="${joint_prefix}wheel_FR_joint" type="continuous">
@@ -249,6 +249,6 @@
       <child link="${link_prefix}wheel_FR_link"/>
       <axis xyz="0 1 0"/>
-      <limit effort="200.0" velocity="20.0"/>
-      <dynamics friction="0.3" damping="0.3"/>
+      <limit effort="800.0" velocity="30.0"/>
+      <dynamics friction="1.0" damping="0.5"/>
     </joint>
     <joint name="${joint_prefix}wheel_RR_joint" type="continuous">
@@ -262,6 +262,6 @@
       <child link="${link_prefix}wheel_RR_link"/>
       <axis xyz="0 1 0"/>
-      <limit effort="200.0" velocity="20.0"/>
-      <dynamics friction="0.3" damping="0.3"/>
+      <limit effort="800.0" velocity="30.0"/>
+      <dynamics friction="1.0" damping="0.5"/>
     </joint>
     <xacro:if value="${default_antenna}">
@@ -492,5 +492,5 @@
         <jointA>rocker_L_joint</jointA>
         <jointB>rocker_R_joint</jointB>
-        <forceConstant>500.0</forceConstant>
+        <forceConstant>2000.0</forceConstant>
       </plugin>
     </gazebo>
@@ -592,8 +592,8 @@
         <odom_topic>${link_prefix}odom</odom_topic>
         <tf_topic>${link_prefix}tf</tf_topic>
-        <max_linear_acceleration>10.0</max_linear_acceleration>
-        <max_angular_acceleration>15.0</max_angular_acceleration>
-        <min_linear_acceleration>-10.0</min_linear_acceleration>
-        <min_angular_acceleration>-15.0</min_angular_acceleration>
+        <max_linear_acceleration>25.0</max_linear_acceleration>
+        <max_angular_acceleration>30.0</max_angular_acceleration>
+        <min_linear_acceleration>-25.0</min_linear_acceleration>
+        <min_angular_acceleration>-30.0</min_angular_acceleration>
       </plugin>
     </gazebo>
